File: BuczekSumowskiSchematics/BuczekMainSchematic.kicad_sch (KiCad schematic)
At the start: 0 parts

Commit message: schematic done
Parts:
- added KILLSWITCH, SW? (x2): SW_DPST_x2, symbol Switch:SW_DPST_x2
- added LipoBattery: 12V, symbol Device:Battery
- added M? (x2): Motor_DC, symbol Motor:Motor_DC
- added R1, R2: 5k, symbol Device:R
- added STAB_3.3V: L78L33_SOT89, Package_TO_SOT_SMD:SOT-89-3, symbol Regulator_Linear:L78L33_SOT89
- added STAB_5V: L78L05_SOT89, Package_TO_SOT_SMD:SOT-89-3, symbol Regulator_Linear:L78L05_SOT89
- added U?: TB6612FNG, Package_SO:SSOP-24_5.3x8.2mm_P0.65mm, symbol Driver_Motor:TB6612FNG
- added U?: IRmodulLineFollower, symbol MyLibrary:IRmodulLineFollower
- added U? (x4): VL53L1CXV0FY1, Sensor_Distance:ST_VL53L1x, symbol Sensor_Distance:VL53L1CXV0FY1
- added U?: YAAJ_BluePill_Part_Like_SWD_Breakout, symbol YAAJ_BluePill_Part_Like_SWD_Breakout:YAAJ_BluePill_Part_Like_SWD_Breakout
- added U?: IRReciever, symbol MyLibrary:IRReciever
Connections:
- new net: M?.1 (+), U?.1 (AO1), U?.2 (AO1)
- new net: U?.10 (PGND2), U?.9 (PGND2)
- new net: M?.1 (+), U?.11 (BO1), U?.12 (BO1)
- new net: U?.15 (PWMB), U?.6 (PA9)
- new net: U?.16 (BIN2), U?.2 (PB13)
- new net: U?.17 (BIN1), U?.3 (PB14)
- new net: U?.21 (AIN1), U?.5 (PA8)
- new net: U?.22 (AIN2), U?.4 (PB15)
- new net: U?.23 (PWMA), U?.7 (PA10)
- new net: M?.2 (-), U?.5 (AO2), U?.6 (AO2)
- new net: M?.2 (-), U?.7 (BO2), U?.8 (BO2)
- new net: U?. (Vcc), U?.10 (PA15)
- new net: U?. (Vcc), U?.11 (PB3)
- new net: U?. (Vcc), U?.8 (PA11)
- new net: U?. (Vcc), U?.9 (PA12)
- new net: KILLSWITCH.1 (A), LipoBattery.2 (-)
- new net: U?.13 (PB5), U?.5 (XSHUT)
- new net: U?. (Vcc), U?.1 (PB12)
- new net: U?.12 (PB4), U?.5 (XSHUT)
- new net: U?.14 (PB6), U?.5 (XSHUT)
- new net: U?.15 (PB7), U?.5 (XSHUT)
- new net +12V: LipoBattery.1 (+), STAB_5V.3 (IN), U?.24 (VM1)
- new net +3.3V: STAB_3.3V.1 (OUT), SW?.1 (A), SW?.3 (A), U?.11 (AVDD), U?.11 (AVDD), U?.11 (AVDD), U?.11 (AVDD), U?.19 (STBY), U?.20 (3V3), U?.20 (VCC)
- new net +5V: STAB_3.3V.3 (IN), STAB_5V.1 (OUT), U?. (Vcc), U?. (Vcc)
- new net GND: KILLSWITCH.2 (B), R1.2, R2.2, STAB_3.3V.2 (GND), STAB_5V.2 (GND), U?. (Vcc), U?. (Vcc), U?.12 (GND), U?.12 (GND), U?.12 (GND), U?.12 (GND), U?.18 (GND), U?.19 (GND), U?.3 (GND), U?.3 (GND), U?.3 (GND), U?.3 (GND), U?.3 (PGND1), U?.4 (GND), U?.4 (GND), U?.4 (GND), U?.4 (GND), U?.4 (PGND1), U?.6 (GND), U?.6 (GND), U?.6 (GND), U?.6 (GND)
- new net SCL1: U?.10 (SCL), U?.10 (SCL), U?.10 (SCL), U?.10 (SCL), U?.16 (PB8)
- new net SDA1: U?.17 (PB9), U?.9 (SDA), U?.9 (SDA), U?.9 (SDA), U?.9 (SDA)
- new net SW1: R1.1, SW?.2 (B), U?.36 (PB11)
- new net SW2: R2.1, SW?.4 (B), U?.35 (PB10)
Other:
- note added: "(Pohled shora) PravoNahore PravoDole LevoDole LevoNahore"
- note added: "Vlevo"
- note added: "Vpravo"
